Commit message: Added b1z1 gym for walking on flat terrain similar to go2. Need to add rewards for arm motion/targets.

File: resources/robots/b1z1/urdf/b1z1_mj.urdf (robot description, URDF)
Before this commit: robot b1z1_description, 39 links, 38 joints
Links:
- removed link ee_gripper_link
- added link world
Joints:
- removed joint ee_gripper
